Commit message: urdf cleanup

File: src/slam_bot_description/models/slam_bot.urdf (robot description, URDF)
Before this commit: robot slam_bot, 5 links, 4 joints
Joints:
- joint base_joint: child base_link -> base_footprint; origin xyz=0.0 0.0 ${(wheel_radius+wheel_zoff)} rpy=0 0 0 -> xyz=0.0 0.0 -${(wheel_radius+wheel_zoff)} rpy=0 0 0; parent base_footprint -> base_link

Commit message: vo K fix

File: src/slam_bot_description/models/slam_bot.urdf (robot description, URDF)
Before this commit: robot slam_bot, 5 links, 4 joints
Joints:
- joint camera_optical_joint: origin xyz=0 0 0 rpy=${-pi/2} 0 ${-pi/2} -> xyz=0 0 0 rpy=${-pi/2} 0 ${+pi/2}

Commit message: reset camera and optical frame to 0

File: src/slam_bot_description/models/slam_bot.urdf (robot description, URDF)
Before this commit: robot slam_bot, 5 links, 4 joints
Joints:
- joint camera_joint: origin xyz=${base_length/2} 0 0 rpy=1.57 0 0 -> xyz=${base_length/2} 0 0 rpy=0 0 0
- joint camera_optical_joint: origin xyz=0 0 0 rpy=${-pi/2} 0 ${+pi/2} -> xyz=0 0 0 rpy=0 0 0

Commit message: vo update , camera link rot 0

File: src/slam_bot_description/models/slam_bot.urdf (robot description, URDF)
Before this commit: robot slam_bot, 5 links, 4 joints
Links:
- link camera_link: geometry collision box size=0.028 0.097 0.0175; visual box size=0.028 0.097 0.0175
Joints:
- joint camera_joint: origin xyz=${base_length/2} 0 0 rpy=1.57 0 0 -> xyz=${base_length/2} 0 0 rpy=0 0 0

Commit message: model update with camera position

File: src/slam_bot_description/models/slam_bot.urdf (robot description, URDF)
Before this commit: robot slam_bot, 5 links, 4 joints
Joints:
- joint camera_joint: origin xyz=${base_length/2} 0 0 rpy=0 0 0 -> xyz=${(base_length/2)+camera_xoff} ${camera_yoff} ${(base_height/2)+camera_zoff} rpy=0 ${-pi/18} 0
- joint camera_optical_joint: origin xyz=0 0 0 rpy=0 0 0 -> xyz=0 -${oak_pro_baseline/2} 0.00465 rpy=${-pi/2} 0 -${pi/2}

Commit message: urdf update for imu link

File: src/slam_bot_description/models/slam_bot.urdf (robot description, URDF)
Before this commit: robot slam_bot, 5 links, 4 joints
Joints:
- joint imu_joint: origin xyz=${base_length/2} 0 0 rpy=0 0 0 -> xyz=0 0 0 rpy=${pi} ${pi} ${pi/2}; parent base_link -> camera_link
